Commit message: updated demo world

File: google_robot/src/resources/description/urdf/model.urdf (robot description, URDF)
Before this commit: robot google_robot, 21 links, 20 joints
Links:
- added link link_left_wheel; collision mesh filename=package://google_robot_description/meshes/converted_link_wh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; visual mesh filename=package://google_robot_description/meshes/converted_link_wh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
- added link link_right_wheel; collision mesh filename=package://google_robot_description/meshes/converted_link_wh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; visual mesh filename=package://google_robot_description/meshes/converted_link_wh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
Joints:
- added joint joint_left_wheel: type continuous, parent base_link, child link_left_wheel, origin xyz=-5.489740642117986e-20 -0.18283 8.563015090875109e-19 rpy=0.0 0.0 1.5707963267948966, axis 0 0 1
- added joint joint_right_wheel: type continuous, parent base_link, child link_right_wheel, origin xyz=-5.489740642117986e-20 0.18283 8.563015090875109e-19 rpy=0.0 0.0 1.5707963267948966, axis 0 0 1

Commit message: update

File: google_robot/src/resources/description/urdf/model.urdf (robot description, URDF)
Before this commit: robot google_robot, 23 links, 22 joints
Links:
- link link_left_wheel: mass None -> 2
- link link_right_wheel: mass None -> 2
Joints:
- joint joint_left_wheel: axis 0 0 1 -> 1 0 0
- joint joint_right_wheel: axis 0 0 1 -> 1 0 0

File: google_robot/src/resources/moveit/config/google_robot.ros2_control.xacro (robot description, xacro)
@@ -18,5 +18,5 @@
             </hardware>
             <joint name="joint_left_wheel">
-                <xacro:if value="${ros2_control_hardware_type == 'mujoco'}">
+                <!-- <xacro:if value="${ros2_control_hardware_type == 'mujoco'}">
                   <param name="position_kp">3000</param>
                   <param name="position_ki">1</param>
@@ -26,11 +26,12 @@
                 </xacro:if>
                 <xacro:unless value="${ros2_control_hardware_type == 'mujoco'}">
-                  <command_interface name="velocity"/>
                 </xacro:unless>
+                 -->
+                <command_interface name="velocity"/>
                 <state_interface name="position"/>
                 <state_interface name="velocity"/>
             </joint>
             <joint name="joint_right_wheel">
-                <xacro:if value="${ros2_control_hardware_type == 'mujoco'}">
+                <!-- <xacro:if value="${ros2_control_hardware_type == 'mujoco'}">
                   <param name="position_kp">3000</param>
                   <param name="position_ki">1</param>
@@ -40,6 +41,6 @@
                 </xacro:if>
                 <xacro:unless value="${ros2_control_hardware_type == 'mujoco'}">
-                  <command_interface name="velocity"/>
-                </xacro:unless>
+                </xacro:unless> -->
+                <command_interface name="velocity"/>
                 <state_interface name="position"/>
                 <state_interface name="velocity"/>
